File: router_backup.kicad_sch (KiCad schematic)
At the start: 21 parts

Commit message: BMS
Parts:
- added C? (x2): C, symbol Device:C
- added D? (x12): 1N4007, Diode_THT:D_DO-41_SOD81_P10.16mm_Horizontal, symbol Diode:1N4007
- added D? (x3): LED, symbol Device:LED
- added J?: Screw_Terminal_01x02, symbol Connector:Screw_Terminal_01x02
- added Q? (x3): BD140, Package_TO_SOT_THT:TO-126-3_Vertical, symbol Transistor_BJT:BD140
- added R? (x6): 20k, symbol Device:R
- added R? (x3): R, symbol Device:R
- added R? (x3): 1k, symbol Device:R
- added R? (x3): 330, symbol Device:R
- added RV? (x3): 20k, symbol Device:R_Potentiometer
- added U? (x3): TL431LP, Package_TO_SOT_THT:TO-92_Inline, symbol Reference_Voltage:TL431LP
- added U? (x2): LM317_TO-220, Package_TO_SOT_THT:TO-220-3_Vertical, symbol Regulator_Linear:LM317_TO-220
- gave numbers to parts that had none: 1
Connections:
- new net: R?.1, R?.2, U?.1 (REF) (x3)
- new net: Q?.3 (B), R?.2, U?.3 (K) (x3)
- new net: R?.1, R?.2, U?.1 (ADJ)
- new net: R?.2, RV?.1 (x3)
- new net: D?.2 (A), Q?.2 (C), R?.1 (x3)
- new net: D?.2 (A), R?.2 (x3)
- new net: D?.1 (K), D?.2 (A) (x9)
- new net: R?.2, U?.2 (VO)
- new net: C?.2, R?.2, U?.2 (VO), U?.3 (VI)
- new net +BATT: C?.1, C?.1, D?.1 (K), D?.1 (K), D?.1 (K), D?.1 (K), D?.1 (K), D?.1 (K), J?.1 (Pin_1), Q?.1 (E), Q?.1 (E), Q?.1 (E), R?.1, R?.1, R?.1, R?.1, R?.1, R?.1, R?.1, R?.1, RV?.2, RV?.2, RV?.2, RV?.3, RV?.3, RV?.3, U?.1 (ADJ), U?.2 (A), U?.2 (A), U?.2 (A)
- new net J1 +: C?.2, J?.2 (Pin_2), U?.3 (VI)

Commit message: added indicator
Parts:
- added D? (x10): LED, symbol Device:LED
- added Q?: IRF9540N, Package_TO_SOT_THT:TO-220-3_Vertical, symbol Transistor_FET:IRF9540N
- added U?: LM3914N, Package_DIP:DIP-18_W7.62mm, symbol Driver_LED:LM3914N
Connections:
- net GND: now also D?.2 (A), D?.2 (A), D?.2 (A), D?.2 (A), D?.2 (A), D?.2 (A), D?.2 (A), D?.2 (A), D?.2 (A), D?.2 (A)
- new net LED1: D?.1 (K), U?.1 (LED1)
- new net LED10: D?.1 (K), U?.10 (LED10)
- new net LED2: D?.1 (K), U?.18 (LED2)
- new net LED3: D?.1 (K), U?.17 (LED3)
- new net LED4: D?.1 (K), U?.16 (LED4)
- new net LED5: D?.1 (K), U?.15 (LED5)
- new net LED6: D?.1 (K), U?.14 (LED6)
- new net LED7: D?.1 (K), U?.13 (LED7)
- new net LED8: D?.1 (K), U?.12 (LED8)
- new net LED9: D?.1 (K), U?.11 (LED9)

Commit message: updated pcb
Parts:
- removed J?: Screw_Terminal_01x02, symbol Connector:Screw_Terminal_01x02
- added D27, D28: 1N5822, Diode_THT:D_DO-201AD_P15.24mm_Horizontal, symbol Diode:1N5822
- added J1: input, TerminalBlock_Phoenix:TerminalBlock_Phoenix_MKDS-1,5-2-5.08_1x02_P5.08mm_Horizontal, symbol Connector:Screw_Terminal_01x02
- added J2: output, TerminalBlock_Phoenix:TerminalBlock_Phoenix_MKDS-1,5-2-5.08_1x02_P5.08mm_Horizontal, symbol Connector:Screw_Terminal_01x02
- added R24: 10k, Resistor_THT:R_Axial_DIN0309_L9.0mm_D3.2mm_P12.70mm_Horizontal, symbol Device:R
- added R25: 56k, Resistor_THT:R_Axial_DIN0309_L9.0mm_D3.2mm_P12.70mm_Horizontal, symbol Device:R
- added R26: R, Resistor_THT:R_Axial_DIN0309_L9.0mm_D3.2mm_P12.70mm_Horizontal, symbol Device:R
- added R27: 4k7, Resistor_THT:R_Axial_DIN0309_L9.0mm_D3.2mm_P12.70mm_Horizontal, symbol Device:R
- added RV5: 10k, Potentiometer_THT:Potentiometer_Bourns_3266Y_Vertical, symbol Device:R_Potentiometer
- 0.03m1: renamed from 0.03m; footprint (none) -> Inductor_SMD:L_6.3x6.3_H3
- C1, C2: renamed from C?; footprint (none) -> Capacitor_THT:C_Radial_D4.0mm_H5.0mm_P1.50mm
- C3: renamed from C?; value C -> 100u; footprint (none) -> Capacitor_THT:C_Radial_D4.0mm_H5.0mm_P1.50mm
- C4, C6: renamed from C?; footprint (none) -> Capacitor_THT:CP_Radial_D4.0mm_P1.50mm
- C5: renamed from C?; value C -> 100u; footprint (none) -> Capacitor_THT:C_Radial_D4.0mm_H7.0mm_P1.50mm
- D10, D16, D17, D18, D19, D20, D21, D22, D23, D24, D25, D26, D5: renamed from D?; footprint (none) -> LED_THT:LED_Rectangular_W3.0mm_H2.0mm
- R1, R10, R11, R12, R13, R14, R15, R16, R17, R18, R19, R2, R20, R21, R22, R23, R3, R4, R5, R6, R7, R8, R9: renamed from R?; footprint (none) -> Resistor_THT:R_Axial_DIN0309_L9.0mm_D3.2mm_P12.70mm_Horizontal
- RV1, RV2, RV3, RV4: renamed from RV?; footprint (none) -> Potentiometer_THT:Potentiometer_Bourns_3266Y_Vertical
- U8: renamed from U?; footprint (none) -> Resistor_THT:R_Array_SIP8
- gave numbers to parts that had none: 26
Connections:
- net J1 + is gone; now on an unnamed net: C5.2, U4.3 (VI)
- net VIN2 is gone; now on net +BATT: R19.2, R22.1, U8.2 (-)
- net +BATT: now also C1.2, C2.2, C4.2, Q3.3 (S), R14.1, R21.1, RV3.1, U1.2 (GND), U5.4 (GND), U8.4 (V-), U9.2 (V-), U9.8 (REFADJ), J1.1 (Pin_1), R24.1, R26.1, R27.2, RV5.3
- net at U9.3 (V+): now also D17.2 (A), D18.2 (A), D19.2 (A), D20.2 (A), D21.2 (A), D22.2 (A), D23.2 (A), D24.2 (A), D25.2 (A), D26.2 (A), Q5.3 (S), U9.9 (MODE), D28.1 (K), R25.1
- net at U9.4 (RLO): now also R26.2
- net at U9.5 (SIG): now also RV5.2
- net at U9.6 (RHI): now also U9.7 (REFOUT), R27.1
- net at Q5.1 (G): now also R24.2
- net at Q5.2 (D): now also D27.2 (A)
- removed net GND: C1.2, C2.2, C4.2, D17.2 (A), D18.2 (A), D19.2 (A), D20.2 (A), D21.2 (A), D22.2 (A), D23.2 (A), D24.2 (A), D25.2 (A), D26.2 (A), Q3.3 (S), R14.1, R21.1, RV3.1, U1.2 (GND), U5.4 (GND), U8.4 (V-)
- net VIN: no longer names the net of R20.2, R21.2, U8.3 (+)
- net VIN: now also D27.1 (K), D28.2 (A), J1.2 (Pin_2)
- new net: R25.2, RV5.1
- new net +: J2.1 (Pin_1)
- new net -: J2.2 (Pin_2)
Other:
- moved on the sheet: Q5, U9
